File: ft4232-indicators.kicad_sch (KiCad schematic)
At the start: 5 parts, among them U1 74HC595D

Commit message: switch to CH344Q
Parts:
- removed D1, D2, D3, D4: LED_Dual_KAK, LED_THT:LED_D5.0mm-3, symbol Device:LED_Dual_KAK
- removed U1: 74HC595D, Package_SO:SO-16_3.9x9.9mm_P1.27mm, symbol 74xx:74HC595
Connections:
- no-connect marks 28 -> 0
Changed lines of the file:
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@@
 (kicad_sch (version 20230121) (generator eeschema)
   (paper "A4")
-  (no_connect (at 88.9 81.28))
-  (no_connect (at 134.62 36.83))
-  (no_connect (at 152.4 71.12))
-  (no_connect (at 154.305 99.06))
-  (no_connect (at 88.9 83.82))
-  (no_connect (at 149.86 39.37))
-  (no_connect (at 68.58 91.44))
-  (no_connect (at 68.58 76.2))
-  (no_connect (at 153.035 122.555))
-  (no_connect (at 68.58 88.9))
-  (no_connect (at 68.58 78.74))
-  (no_connect (at 149.86 34.29))
-  (no_connect (at 68.58 86.36))
-  (no_connect (at 88.9 76.2))
-  (no_connect (at 68.58 81.28))
-  (no_connect (at 78.74 71.12))
-  (no_connect (at 68.58 93.98))
-  (no_connect (at 88.9 88.9))
-  (no_connect (at 68.58 99.06))
-  (no_connect (at 137.795 125.095))
-  (no_connect (at 154.305 93.98))
-  (no_connect (at 68.58 83.82))
-  (no_connect (at 137.16 68.58))
-  (no_connect (at 153.035 127.635))
-  (no_connect (at 139.065 96.52))
-  (no_connect (at 78.74 104.14))
-  (no_connect (at 152.4 66.04))
-  (no_connect (at 88.9 91.44))
-  (symbol (lib_id "Device:LED_Dual_KAK") (at 142.24 36.83 0) (unit 1)
-    (in_bom yes) (on_board yes) (dnp no) (fields_autoplaced)
-    (property "Reference" "D1" (at 142.3035 25.4 0)
-      (effects (font (size 1.27 1.27)))
-    )
-    (property "Value" "LED_Dual_KAK" (at 142.3035 27.94 0)
-      (effects (font (size 1.27 1.27)))
-    )
-    (property "Footprint" "LED_THT:LED_D5.0mm-3" (at 143.51 36.83 0)
-      (effects (font (size 1.27 1.27)) hide)
-    )
-    (property "Datasheet" "~" (at 143.51 36.83 0)
-      (effects (font (size 1.27 1.27)) hide)
-    )
-    (pin "1")
-    (pin "2")
-    (pin "3")
-    (instances
-      (project "isouart4"
-        (path "/7c54d849-3d49-4f8e-b560-9dd1d738085c"
-          (reference "D1") (unit 1)
-        )
-        (path "/7c54d849-3d49-4f8e-b560-9dd1d738085c/2d235b8c-e233-4472-a8af-47eb53407ee3"
-          (reference "D1") (unit 1)
-        )
-        (path "/7c54d849-3d49-4f8e-b560-9dd1d738085c/cd7e2163-e08f-4cc8-b5c0-cec347de14ac"
-          (reference "D1") (unit 1)
-        )
-      )
-    )
-  )
-  (symbol (lib_id "Device:LED_Dual_KAK") (at 146.685 96.52 0) (unit 1)
-    (in_bom yes) (on_board yes) (dnp no) (fields_autoplaced)
-    (property "Reference" "D4" (at 146.7485 85.09 0)
-      (effects (font (size 1.27 1.27)))
-    )
-    (property "Value" "LED_Dual_KAK" (at 146.7485 87.63 0)
-      (effects (font (size 1.27 1.27)))
-    )
-    (property "Footprint" "LED_THT:LED_D5.0mm-3" (at 147.955 96.52 0)
-      (effects (font (size 1.27 1.27)) hide)
-    )
-    (property "Datasheet" "~" (at 147.955 96.52 0)
-      (effects (font (size 1.27 1.27)) hide)
-    )
-    (pin "1")
-    (pin "2")
-    (pin "3")
-    (instances
-      (project "isouart4"
-        (path "/7c54d849-3d49-4f8e-b560-9dd1d738085c"
-          (reference "D4") (unit 1)
-        )
-        (path "/7c54d849-3d49-4f8e-b560-9dd1d738085c/2d235b8c-e233-4472-a8af-47eb53407ee3"
-          (reference "D4") (unit 1)
-        )
-        (path "/7c54d849-3d49-4f8e-b560-9dd1d738085c/cd7e2163-e08f-4cc8-b5c0-cec347de14ac"
-          (reference "D4") (unit 1)
-        )
-      )
-    )
-  )
-  (symbol (lib_id "74xx:74HC595") (at 78.74 86.36 0) (mirror y) (unit 1)
-    (in_bom yes) (on_board yes) (dnp no)
-    (property "Reference" "U1" (at 76.5459 68.58 0)
-      (effects (font (size 1.27 1.27)) (justify left))
-    )
-    (property "Value" "74HC595D" (at 76.5459 71.12 0)
-      (effects (font (size 1.27 1.27)) (justify left))
-    )
-    (property "Footprint" "Package_SO:SO-16_3.9x9.9mm_P1.27mm" (at 78.74 86.36 0)
-      (effects (font (size 1.27 1.27)) hide)
-    )
-    (property "Datasheet" "http://www.ti.com/lit/ds/symlink/sn74hc595.pdf" (at 78.74 86.36 0)
-      (effects (font (size 1.27 1.27)) hide)
-    )
-    (pin "1")
-    (pin "10")
-    (pin "11")
-    (pin "12")
-    (pin "13")
-    (pin "14")
-    (pin "15")
-    (pin "16")
-    (pin "2")
-    (pin "3")
-    (pin "4")
-    (pin "5")
-    (pin "6")
-    (pin "7")
-    (pin "8")
-    (pin "9")
-    (instances
-      (project "isouart4"
-        (path "/7c54d849-3d49-4f8e-b560-9dd1d738085c"
-          (reference "U1") (unit 1)
-        )
-        (path "/7c54d849-3d49-4f8e-b560-9dd1d738085c/2d235b8c-e233-4472-a8af-47eb53407ee3"
-          (reference "U1") (unit 1)
-        )
-        (path "/7c54d849-3d49-4f8e-b560-9dd1d738085c/cd7e2163-e08f-4cc8-b5c0-cec347de14ac"
-          (reference "U5") (unit 1)
-        )
-      )
-    )
-  )
-  (symbol (lib_id "Device:LED_Dual_KAK") (at 144.78 68.58 0) (unit 1)
-    (in_bom yes) (on_board yes) (dnp no) (fields_autoplaced)
-    (property "Reference" "D2" (at 144.8435 57.15 0)
-      (effects (font (size 1.27 1.27)))
-    )
-    (property "Value" "LED_Dual_KAK" (at 144.8435 59.69 0)
-      (effects (font (size 1.27 1.27)))
-    )
-    (property "Footprint" "LED_THT:LED_D5.0mm-3" (at 146.05 68.58 0)
-      (effects (font (size 1.27 1.27)) hide)
-    )
-    (property "Datasheet" "~" (at 146.05 68.58 0)
-      (effects (font (size 1.27 1.27)) hide)
-    )
-    (pin "1")
-    (pin "2")
-    (pin "3")
-    (instances
-      (project "isouart4"
-        (path "/7c54d849-3d49-4f8e-b560-9dd1d738085c"
-          (reference "D2") (unit 1)
-        )
-        (path "/7c54d849-3d49-4f8e-b560-9dd1d738085c/2d235b8c-e233-4472-a8af-47eb53407ee3"
-          (reference "D2") (unit 1)
-        )
-        (path "/7c54d849-3d49-4f8e-b560-9dd1d738085c/cd7e2163-e08f-4cc8-b5c0-cec347de14ac"
-          (reference "D2") (unit 1)
-        )
-      )
-    )
-  )
-  (symbol (lib_id "Device:LED_Dual_KAK") (at 145.415 125.095 0) (unit 1)
-    (in_bom yes) (on_board yes) (dnp no) (fields_autoplaced)
-    (property "Reference" "D3" (at 145.4785 113.665 0)
-      (effects (font (size 1.27 1.27)))
-    )
-    (property "Value" "LED_Dual_KAK" (at 145.4785 116.205 0)
-      (effects (font (size 1.27 1.27)))
-    )
-    (property "Footprint" "LED_THT:LED_D5.0mm-3" (at 146.685 125.095 0)
-      (effects (font (size 1.27 1.27)) hide)
-    )
-    (property "Datasheet" "~" (at 146.685 125.095 0)
-      (effects (font (size 1.27 1.27)) hide)
-    )
-    (pin "1")
-    (pin "2")
-    (pin "3")
-    (instances
-      (project "isouart4"
-        (path "/7c54d849-3d49-4f8e-b560-9dd1d738085c"
-          (reference "D3") (unit 1)
-        )
-        (path "/7c54d849-3d49-4f8e-b560-9dd1d738085c/2d235b8c-e233-4472-a8af-47eb53407ee3"
-          (reference "D3") (unit 1)
-        )
-        (path "/7c54d849-3d49-4f8e-b560-9dd1d738085c/cd7e2163-e08f-4cc8-b5c0-cec347de14ac"
-          (reference "D3") (unit 1)
-        )
-      )
-    )
-  )
 )
