File: isouart4.kicad_pcb (KiCad board)
At the start: 2 copper layers, 89 x 99 mm, 83 parts, among them J1 USB_B, J2 Conn_01x04, J3 Conn_01x04, J4 Conn_01x04, J5 Conn_01x04, U1 AMS1117-3.3, U10 74HC123, U11 74HC123, U2 π122U31, U3 π122U31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

Commit message: Fix xtal 7050 footprint warning by creating isouart4 footprint copy
Parts:
- Y1: footprint Crystal:Crystal_SMD_7050-4Pin_7.0x5.0mm -> isouart4:Crystal_SMD_7050-4Pin_7.0x5.0mm
Changed lines of the file:
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@@
     )
   )
-  (footprint "Crystal:Crystal_SMD_7050-4Pin_7.0x5.0mm" (layer "B.Cu")
+  (footprint "isouart4:Crystal_SMD_7050-4Pin_7.0x5.0mm" (layer "B.Cu")
     (at 170.625 104.675 45)
     (descr "SMD Crystal SERIES SMD7050/4 https://www.foxonline.com/pdfs/FQ7050.pdf, 7.0x5.0mm^2 package")
@@
     (property "ki_keywords" "quartz ceramic resonator oscillator")
     (attr smd)
-    (fp_text reference "Y1" (at 0 3.7 45) (layer "B.SilkS")
+    (fp_text reference "Y1" (at 0 3.7 225) (layer "B.SilkS")
         (effects (font (size 1 1) (thickness 0.15)) (justify mirror))
     )
-    (fp_text value "8MHz" (at 0 -3.7 45) (layer "B.Fab")
+    (fp_text value "8MHz" (at 0 -3.7 225) (layer "B.Fab")
         (effects (font (size 1 1) (thickness 0.15)) (justify mirror))
     )
-    (fp_text user "${REFERENCE}" (at 0 0 45) (layer "B.Fab")
+    (fp_text user "${REFERENCE}" (at 0 0 225) (layer "B.Fab")
         (effects (font (size 1 1) (thickness 0.15)) (justify mirror))
     )

Commit message: Fix FB footprint warning by creating isouart4 footprint copy
Parts:
- L1, L2, L3: footprint Inductor_SMD:L_TDK_NLV25_2.5x2.0mm -> isouart4:FB_0805_2012Metric
Changed lines of the file:
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@@
     )
   )
-  (footprint "Inductor_SMD:L_TDK_NLV25_2.5x2.0mm" (layer "B.Cu")
+  (footprint "isouart4:FB_0805_2012Metric" (layer "B.Cu")
     (at 152.665 85.82 90)
     (descr "TDK NLV25, 2.5x2.0x1.8mm, https://product.tdk.com/info/en/catalog/datasheets/inductor_commercial_standard_nlv25-ef_en.pdf")
@@
     (property "ki_keywords" "inductor choke coil reactor magnetic")
     (attr smd)
-    (fp_text reference "L1" (at 0 3.275 90) (layer "B.SilkS")
-        (effects (font (size 1 1) (thickness 0.15)) (justify mirror))
-    )
-    (fp_text value "L_Ferrite_Small" (at 0 -2 90) (layer "B.Fab")
-        (effects (font (size 1 1) (thickness 0.15)) (justify mirror))
-    )
-    (fp_text user "${REFERENCE}" (at 0 0 90) (layer "B.Fab")
+    (fp_text reference "L1" (at 0 2 270) (layer "B.SilkS")
+        (effects (font (size 1 1) (thickness 0.15)) (justify mirror))
+    )
+    (fp_text value "L_Ferrite_Small" (at 0 -2 270) (layer "B.Fab")
+        (effects (font (size 1 1) (thickness 0.15)) (justify mirror))
+    )
+    (fp_text user "${REFERENCE}" (at 0 0 270) (layer "B.Fab")
         (effects (font (size 0.5 0.5) (thickness 0.08)) (justify mirror))
     )
@@
     )
   )
-  (footprint "Inductor_SMD:L_TDK_NLV25_2.5x2.0mm" (layer "B.Cu")
+  (footprint "isouart4:FB_0805_2012Metric" (layer "B.Cu")
     (at 157.8 121.3 -90)
     (descr "TDK NLV25, 2.5x2.0x1.8mm, https://product.tdk.com/info/en/catalog/datasheets/inductor_commercial_standard_nlv25-ef_en.pdf")
@@
     (property "ki_keywords" "inductor choke coil reactor magnetic")
     (attr smd)
-    (fp_text reference "L2" (at -3.24 -0.15 90) (layer "B.SilkS")
+    (fp_text reference "L2" (at 1.93 -2.34 90) (layer "B.SilkS")
         (effects (font (size 1 1) (thickness 0.15)) (justify mirror))
     )
@@
     )
   )
-  (footprint "Inductor_SMD:L_TDK_NLV25_2.5x2.0mm" (layer "B.Cu")
+  (footprint "isouart4:FB_0805_2012Metric" (layer "B.Cu")
     (at 177.425 107.2 45)
     (descr "TDK NLV25, 2.5x2.0x1.8mm, https://product.tdk.com/info/en/catalog/datasheets/inductor_commercial_standard_nlv25-ef_en.pdf")
@@
     (property "ki_keywords" "inductor choke coil reactor magnetic")
     (attr smd)
-    (fp_text reference "L3" (at 0 2 45) (layer "B.SilkS")
-        (effects (font (size 1 1) (thickness 0.15)) (justify mirror))
-    )
-    (fp_text value "L_Ferrite_Small" (at 0 -2 45) (layer "B.Fab")
-        (effects (font (size 1 1) (thickness 0.15)) (justify mirror))
-    )
-    (fp_text user "${REFERENCE}" (at 0 0 45) (layer "B.Fab")
-        (effects (font (size 0.5 0.5) (thickness 0.08)) (justify mirror))
-    )
+    (fp_text reference "L3" (at 0 2 225) (layer "B.SilkS")
+        (effects (font (size 1 1) (thickness 0.15)) (justify mirror))
+    )
+    (fp_text value "L_Ferrite_Small" (at 0 -2 225) (layer "B.Fab")
+        (effects (font (size 1 1) (thickness 0.15)) (justify mirror))
+    )
+    (fp_text user "${REFERENCE}" (at 0 0 225) (layer "B.Fab")
+        (effects (font (size 0.5 0.5) (thickness 0.08)) (justify mirror))
+    )
