File: isouart4.kicad_sch (KiCad schematic)
At the start: 25 parts, among them J1 USB_B, J2 Conn_01x04, J3 Conn_01x04, J4 Conn_01x04, J5 Conn_01x04, U2 π122U31, U3 AMS1117-3.3, U4 π122U31, U5 π122U31, U6 π122U31

Commit message: reannotate
Parts:
- renumbered C2 to C1, C7 to C2, U3 to U1, U6 to U2, U2 to U3

Commit message: Fix FB footprint warning by creating isouart4 footprint copy
Parts:
- L1, L2: footprint Inductor_SMD:L_TDK_NLV25_2.5x2.0mm -> isouart4:FB_0805_2012Metric; symbol Device:L_Ferrite_Small -> isouart4:L_Ferrite_Small
Changed lines of the file:
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@@
     )
   )
-  (symbol (lib_id "Device:L_Ferrite_Small") (at 86.36 88.9 90) (unit 1)
+  (symbol (lib_id "isouart4:L_Ferrite_Small") (at 86.36 88.9 90) (unit 1)
     (in_bom yes) (on_board yes) (dnp no) (fields_autoplaced)
     (property "Reference" "L1" (at 86.36 82.55 90)
@@
       (effects (font (size 1.27 1.27)))
     )
-    (property "Footprint" "Inductor_SMD:L_TDK_NLV25_2.5x2.0mm" (at 86.36 88.9 0)
+    (property "Footprint" "isouart4:FB_0805_2012Metric" (at 86.36 88.9 0)
       (effects (font (size 1.27 1.27)) hide)
     )
@@
     )
   )
-  (symbol (lib_id "Device:L_Ferrite_Small") (at 86.995 143.51 90) (unit 1)
+  (symbol (lib_id "isouart4:L_Ferrite_Small") (at 86.995 143.51 90) (unit 1)
     (in_bom yes) (on_board yes) (dnp no) (fields_autoplaced)
     (property "Reference" "L2" (at 86.995 137.16 90)
@@
       (effects (font (size 1.27 1.27)))
     )
-    (property "Footprint" "Inductor_SMD:L_TDK_NLV25_2.5x2.0mm" (at 86.995 143.51 0)
-      (effects (font (size 1.27 1.27)) hide)
-    )
+    (property "Footprint" "isouart4:FB_0805_2012Metric" (at 86.995 143.51 0)
+      (effects (font (size 1.27 1.27)) hide)
+    )
