File: indicators-ch1.kicad_sch (KiCad schematic)
At the start: 2 parts, among them U10 74HC123

Commit message: Flush
Parts:
- added C13, C17, C21: 1uF, Capacitor_SMD:C_0805_2012Metric_Pad1.18x1.45mm_HandSolder, symbol Device:C_Small
- added R3 (x2): 1k, Resistor_SMD:R_0805_2012Metric_Pad1.20x1.40mm_HandSolder, symbol Device:R_Small
- added R3 (x2): 220k, Resistor_SMD:R_0805_2012Metric_Pad1.20x1.40mm_HandSolder, symbol Device:R_Small
Connections:
- net V+MON: now reaches U10.16 (VCC)
- net V+MON: now also D5.2 (A), U10.10 (B), U10.11 (Clr), U10.2 (B), U10.3 (Clr), C21.2, R3.1, R3.1
- net GNDMON: now reaches U10.8 (GND)
- net GNDMON: now also C21.1
- net at D5.1 (K1): now also R3.1
- net at D5.3 (K2): now also R3.1
- net TXMON: now reaches U10.1 (A)
- net at U10.14 (Cext): now also C17.1
- net at U10.15 (RCext): now also C17.2, R3.2
- net at U10.4 (~{Q}): now also R3.2
- net at U10.12 (~{Q}): now also R3.2
- net at U10.6 (Cext): now also C13.1
- net at U10.7 (RCext): now also C13.2, R3.2
- net RXMON: now reaches U10.9 (A)
- no-connect marks 19 -> 2
Other:
- moved on the sheet: D5, U10A, U10B, U10C

Commit message: Flush latest changes
Parts:
- C21: value 1uF -> 100n
Changed lines of the file:
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@@
       (effects (font (size 1.27 1.27)))
     )
-    (property "Value" "1uF" (at 203.2 90.805 90)
+    (property "Value" "100n" (at 203.2 90.805 90)
       (effects (font (size 1.27 1.27)))
     )

Commit message: reannotate
Parts:
- renumbered C17 to C18, C13 to C19, C21 to C20

Commit message: adjust silkscreen and led positions; reannotate
Parts:
- renumbered C18 to C20, C19 to C21, C20 to C22
Changed lines of the file:
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@@
   (symbol (lib_id "Device:C_Small") (at 90.17 108.585 180) (unit 1)
     (in_bom yes) (on_board yes) (dnp no)
-    (property "Reference" "C18" (at 85.09 109.855 0)
+    (property "Reference" "C20" (at 85.09 109.855 0)
       (effects (font (size 1.27 1.27)))
     )
@@
       (project "isouart4"
         (path "/7c54d849-3d49-4f8e-b560-9dd1d738085c/958710c5-0600-4104-a764-b45629adc817"
-          (reference "C18") (unit 1)
-        )
-        (path "/7c54d849-3d49-4f8e-b560-9dd1d738085c/80cea6f2-87b4-4a40-8c2f-e4524d3d8e29"
-          (reference "C21") (unit 1)
-        )
-        (path "/7c54d849-3d49-4f8e-b560-9dd1d738085c/b1d70d56-3a6d-4a09-94ea-3708cca9e5ca"
-          (reference "C24") (unit 1)
-        )
-        (path "/7c54d849-3d49-4f8e-b560-9dd1d738085c/4a921ac0-5400-4f95-9340-83876c5a92c2"
-          (reference "C27") (unit 1)
+          (reference "C20") (unit 1)
+        )
+        (path "/7c54d849-3d49-4f8e-b560-9dd1d738085c/80cea6f2-87b4-4a40-8c2f-e4524d3d8e29"
+          (reference "C23") (unit 1)
+        )
+        (path "/7c54d849-3d49-4f8e-b560-9dd1d738085c/b1d70d56-3a6d-4a09-94ea-3708cca9e5ca"
+          (reference "C26") (unit 1)
+        )
+        (path "/7c54d849-3d49-4f8e-b560-9dd1d738085c/4a921ac0-5400-4f95-9340-83876c5a92c2"
+          (reference "C29") (unit 1)
         )
       )
@@
   (symbol (lib_id "Device:C_Small") (at 203.2 96.52 270) (unit 1)
     (in_bom yes) (on_board yes) (dnp no)
-    (property "Reference" "C20" (at 203.835 92.71 90)
+    (property "Reference" "C22" (at 203.835 92.71 90)
       (effects (font (size 1.27 1.27)))
     )
@@
       (project "isouart4"
         (path "/7c54d849-3d49-4f8e-b560-9dd1d738085c/958710c5-0600-4104-a764-b45629adc817"
-          (reference "C20") (unit 1)
-        )
-        (path "/7c54d849-3d49-4f8e-b560-9dd1d738085c/80cea6f2-87b4-4a40-8c2f-e4524d3d8e29"
-          (reference "C23") (unit 1)
-        )
-        (path "/7c54d849-3d49-4f8e-b560-9dd1d738085c/b1d70d56-3a6d-4a09-94ea-3708cca9e5ca"
-          (reference "C26") (unit 1)
-        )
-        (path "/7c54d849-3d49-4f8e-b560-9dd1d738085c/4a921ac0-5400-4f95-9340-83876c5a92c2"
-          (reference "C29") (unit 1)
+          (reference "C22") (unit 1)
+        )
+        (path "/7c54d849-3d49-4f8e-b560-9dd1d738085c/80cea6f2-87b4-4a40-8c2f-e4524d3d8e29"
+          (reference "C25") (unit 1)
+        )
+        (path "/7c54d849-3d49-4f8e-b560-9dd1d738085c/b1d70d56-3a6d-4a09-94ea-3708cca9e5ca"
+          (reference "C28") (unit 1)
+        )
+        (path "/7c54d849-3d49-4f8e-b560-9dd1d738085c/4a921ac0-5400-4f95-9340-83876c5a92c2"
+          (reference "C31") (unit 1)
         )
       )
@@
   (symbol (lib_id "Device:C_Small") (at 140.335 108.585 180) (unit 1)
     (in_bom yes) (on_board yes) (dnp no)
-    (property "Reference" "C19" (at 135.255 109.855 0)
+    (property "Reference" "C21" (at 135.255 109.855 0)
       (effects (font (size 1.27 1.27)))
     )
@@
       (project "isouart4"
         (path "/7c54d849-3d49-4f8e-b560-9dd1d738085c/958710c5-0600-4104-a764-b45629adc817"
-          (reference "C19") (unit 1)
-        )
-        (path "/7c54d849-3d49-4f8e-b560-9dd1d738085c/80cea6f2-87b4-4a40-8c2f-e4524d3d8e29"
-          (reference "C22") (unit 1)
-        )
-        (path "/7c54d849-3d49-4f8e-b560-9dd1d738085c/b1d70d56-3a6d-4a09-94ea-3708cca9e5ca"
-          (reference "C25") (unit 1)
-        )
-        (path "/7c54d849-3d49-4f8e-b560-9dd1d738085c/4a921ac0-5400-4f95-9340-83876c5a92c2"
-          (reference "C28") (unit 1)
-        )
-      )
+          (reference "C21") (unit 1)
+        )
+        (path "/7c54d849-3d49-4f8e-b560-9dd1d738085c/80cea6f2-87b4-4a40-8c2f-e4524d3d8e29"
+          (reference "C24") (unit 1)
+        )
+        (path "/7c54d849-3d49-4f8e-b560-9dd1d738085c/b1d70d56-3a6d-4a09-94ea-3708cca9e5ca"
+          (reference "C27") (unit 1)
+        )
+        (path "/7c54d849-3d49-4f8e-b560-9dd1d738085c/4a921ac0-5400-4f95-9340-83876c5a92c2"
+          (reference "C30") (unit 1)
+        )
+      )

Commit message: Add some title text to the schematic sheets
Other:
- note added: "UART TX/RX Indicator"
- title: (none) -> Galvanically Isolated USB attached Quad UART
Changed lines of the file:
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@@
 (kicad_sch (version 20230121) (generator eeschema)
   (paper "A4")
+  (title_block
+    (title "Galvanically Isolated USB attached Quad UART")
+  )
   (junction (at 140.335 106.045) (diameter 0) (color 0 0 0 0)
   )
@@
     (stroke (width 0) (type default))
   )
+  (text "UART TX/RX Indicator" (at 182.245 175.895 0)
+    (effects (font (size 3 3) (thickness 0.6) bold) (justify left bottom))
+  )
   (hierarchical_label "RXMON" (shape input) (at 144.78 116.205 180) (fields_autoplaced)
